File: csi_passthrough_board/csi_passthrough_board.kicad_pcb (KiCad board)
At the start: 4 copper layers, 130 x 149 mm, 19 parts, among them J1 CSI-22-F32Q-1A7H1-11022, J10 Screw_Terminal_01x05, J101 CSI-22-F32Q-1A7H1-11022, J102 CSI-22-F32Q-1A7H1-11022, J103 CSI-22-F32Q-1A7H1-11022, J104 CSI-22-F32Q-1A7H1-11022, J105 CSI-22-F32Q-1A7H1-11022, J106 CSI-22-F32Q-1A7H1-11022, J107 CSI-22-F32Q-1A7H1-11022, J108 CSI-22-F32Q-1A7H1-11022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

Commit message: after standoffs, before shifting
Parts:
- added MP1: M2.5 x 3.5mm, WA-SMSI_9774XXX151:WA-SMSI_9774035151, B.Cu at (121.1, 44.3)
- added MP2: M2.5 x 3.5mm, WA-SMSI_9774XXX151:WA-SMSI_9774035151, B.Cu at (121.1, 144.7)
- added MP3: M2.5 x 3.5mm, WA-SMSI_9774XXX151:WA-SMSI_9774035151, B.Cu at (221.5, 44.3)
- added MP4: M2.5 x 3.5mm, WA-SMSI_9774XXX151:WA-SMSI_9774035151, B.Cu at (221.5, 144.7)
- moved J10 54.5 mm to (238.4, 86.6), turned to 90 degrees
- moved U1 21.7 mm to (142.9, 102.6)
- moved J101 21.7 mm to (211.3, 129.3)
- moved J102 21.7 mm to (191.8, 129.3)
- moved J103 21.7 mm to (182.3, 109.0)
- moved J104 21.7 mm to (182.3, 89.0)
- moved J107 21.7 mm to (121.5, 117.5)
- moved J108 21.7 mm to (121.5, 97.0)
- moved J2 21.7 mm to (221.3, 94.5)
- moved J4 21.7 mm to (121.3, 94.5)
- moved J5 21.7 mm to (201.3, 64.5)
- moved J6 21.7 mm to (201.3, 124.5)
- moved J7 21.7 mm to (141.3, 124.5)
- moved J8 21.7 mm to (141.3, 64.5)
- moved U2 21.7 mm to (202.7, 94.1)
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Routing:
- net /SDA: track 144.5 -> 104.0 mm
- net +3V3: track 155.0 -> 116.0 mm
- net +5V: track 155.2 -> 116.7 mm
- net /SCL: track 137.5 -> 102.7 mm, vias 0 -> 1
- net /CAM1-SDA: track 149.7 -> 148.2 mm
- net /CAM1-VCC: track 153.0 -> 151.6 mm
- net /CAM1-SCL: track 145.6 -> 144.6 mm
- net /CAM1-POWER-EN: track 139.1 -> 138.4 mm
- net /CAM1-LED-EN: track 142.3 -> 141.8 mm
Other:
- board size 130 x 149 mm -> 148.5 x 148.3 mm
- board text added: "CSI Pass-Through Board V1.2"
- board text removed: "CSI Pass-Through Board V1.1"
