File: csi_passthrough_board/csi_passthrough_board.kicad_sch (KiCad schematic)
At the start: 19 parts, among them J1 CSI-22-F32Q-1A7H1-11022, J10 Screw_Terminal_01x05, J101 CSI-22-F32Q-1A7H1-11022, J102 CSI-22-F32Q-1A7H1-11022, J103 CSI-22-F32Q-1A7H1-11022, J104 CSI-22-F32Q-1A7H1-11022, J105 CSI-22-F32Q-1A7H1-11022, J106 CSI-22-F32Q-1A7H1-11022, J107 CSI-22-F32Q-1A7H1-11022, J108 CSI-22-F32Q-1A7H1-11022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

Commit message: after standoffs, before shifting
Parts:
- added MP1, MP2, MP3, MP4: M2.5 x 3.5mm, WA-SMSI_9774XXX151:WA-SMSI_9774035151, symbol WA-SMSI_9774XXX151:WA-SMSI_9774XXX151
