File: csi_passthrough_board/csi_passthrough_board.kicad_sch (KiCad schematic)
At the start: 23 parts, among them J1 CSI-22-F32Q-1A7H1-11022, J10 Screw_Terminal_01x05, J101 CSI-22-F32Q-1A7H1-11022, J102 CSI-22-F32Q-1A7H1-11022, J103 CSI-22-F32Q-1A7H1-11022, J104 CSI-22-F32Q-1A7H1-11022, J105 CSI-22-F32Q-1A7H1-11022, J106 CSI-22-F32Q-1A7H1-11022, J107 CSI-22-F32Q-1A7H1-11022, J108 CSI-22-F32Q-1A7H1-11022, J2 CSI-22-F32Q-1A7H1-11022, J3 CSI-22-F32Q-1A7H1-11022, J4 CSI-22-F32Q-1A7H1-11022, J5 CSI-22-F32Q-1A7H1-11022, J6 CSI-22-F32Q-1A7H1-11022, J7 CSI-22-F32Q-1A7H1-11022, J8 CSI-22-F32Q-1A7H1-11022

Commit message: V1.4, added bottom entry pins
Parts:
- removed U1, U2: (no value), lachs_lib:CSI_Mux_Hat, symbol lachs_lib:CSI_Mux_Hat
- added J11, J9: M20-7810345, M20_7810345:HARWIN_M20-7810345, symbol M20-7810345:M20-7810345
- added MP10, MP5, MP6, MP7, MP8, MP9: M2.5 x 4mm, 9774040151R:WA-SMSI_9774040151, symbol WA-SMSI_9774XXX151:WA-SMSI_9774XXX151
- added U1, U2: CSI Mux Hat, CSI_Mux_hat:CSI_Mux_Hat, symbol csi_mux_hat:CSI_Mux_Hat
- J1, J101, J102, J103, J104, J105, J106, J107, J108, J2, J3, J4, J5, J6, J7, J8: footprint lachs_lib:AMPHENOL_F32Q-1A7H1-11022 -> F32Q_1A7H1_11022:AMPHENOL_F32Q-1A7H1-11022
- MP1, MP2, MP3, MP4: value M2.5 x 3.5mm -> M2.5 x 12mm; footprint WA-SMSI_9774XXX151:WA-SMSI_9774035151 -> 9774120360R:WA-SMSI_9774120360; DATASHEET-URL https://www.we-online.com/catalog/datasheet/9774035151R.pdf -> https://www.we-online.com/catalog/datasheet/9774040151R.pdf; PART-NUMBER 9774035151R -> 9774040151R; PIN-LENGTH 3.5mm -> 4mm
Connections:
- net +3V3: now also J10.1 (Pin_1), J11.5, J9.5; no longer J10.5 (Pin_5)
- net +5V: now also J10.2 (Pin_2), J11.4, J11.6, J9.4, J9.6; no longer J10.4 (Pin_4)
- net GND: now also J10.5 (Pin_5), J11.2, J9.2; no longer J10.1 (Pin_1)
- net SCL: now also J10.4 (Pin_4), J11.1, J9.1; no longer J10.2 (Pin_2)
- net SDA: now also J11.3, J9.3
- no-connect marks 80 -> 90
Other:
- moved on the sheet: J1, J10, J101, J102, J103, J104, J105, J106, J107, J108, J2, J3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

Commit message: production v1_4
Parts:
- J1, J101, J102, J103, J104, J105, J106, J107, J108, J2, J3, J4, J5, J6, J7, J8: LCSC Part # (none) -> C3169253
- J10: now not fitted; now left out of the parts list
- J11, J9: LCSC Part # (none) -> C5666544
- MP1, MP2, MP3, MP4: LCSC Part # (none) -> C22431359
- MP10, MP5, MP6, MP7, MP8, MP9: LCSC Part # (none) -> C5182034
- U1, U2: now not fitted
